File: main_board/openautolab.kicad_pcb (KiCad board)
At the start: 2 copper layers, 98 x 84 mm, 63 parts, among them J1 GP7, J10 FILTER_PUMP, J11 FILTER_SENSOR, J12 PWR_IN, J13 HX711, J14 SERVO, J15 Display, J2 GP6, J3 GP5, J4 GP4, J5 GP3, J6 GP2, J7 GP1, J8 GP0, J9 PUMP, Q1 TSM2302CX, Q2 TSM2302CX, Q3 TSM2302CX, Q4 TSM2302CX, Q5 TSM2302CX, Q6 TSM2302CX, Q7 TSM2302CX, Q8 TSM2302CX, Q9 TSM2302CX, SW0 GP20, SW1 GP21, SW2 GP22, SW3 SW_DPST_x2, U2 LM2575-5.0BT, U3 Pico, U4 A4950E

Commit message: prepare for routing
Parts:
- added NT1: NetTie_2, NetTie:NetTie-2_SMD_Pad0.5mm, F.Cu at (109.5, 80.5)
Connections:
- C1 pad 2: GND -> GNDPWR
- C3 pad 2: GND -> GNDPWR
- J12 pad 1: GND -> GNDPWR
- Q1 pad 2: GND -> GNDPWR
- Q2 pad 2: GND -> GNDPWR
- Q3 pad 2: GND -> GNDPWR
- Q4 pad 2: GND -> GNDPWR
- Q5 pad 2: GND -> GNDPWR
- Q6 pad 2: GND -> GNDPWR
- Q7 pad 2: GND -> GNDPWR
- Q8 pad 2: GND -> GNDPWR
- Q9 pad 2: GND -> GNDPWR
- R10 pad 2: GND -> GNDPWR
- R12 pad 2: GND -> GNDPWR
- R14 pad 2: GND -> GNDPWR
- R16 pad 2: GND -> GNDPWR
- R18 pad 2: GND -> GNDPWR
- R2 pad 2: GND -> GNDPWR
- R4 pad 2: GND -> GNDPWR
- R6 pad 2: GND -> GNDPWR
- R8 pad 2: GND -> GNDPWR
- U2 pad 3: GND -> GNDPWR
- U2 pad 5: GND -> GNDPWR
- U4 pad 1: GND -> GNDPWR
- U4 pad 9: GND -> GNDPWR
Changed lines of the file:
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@@
 	(net 68 "unconnected-(U3-VBUS-Pad40)")
 	(net 69 "unconnected-(U3-GPIO13-Pad17)")
+	(net 70 "GNDPWR")
+	(footprint "NetTie:NetTie-2_SMD_Pad0.5mm"
+		(layer "F.Cu")
+		(at 109.5 80.5 180)
+		(descr "Net tie, 2 pin, 0.5mm square SMD pads")
+		(tags "net tie")
+		(property "Reference" "NT1"
+			(at 0 -1.2 360)
+			(layer "F.SilkS")
+			(hide yes)
+			(effects
+				(font
+					(size 1 1)
+					(thickness 0.15)
+				)
+			)
+		)
+		(property "Value" "NetTie_2"
+			(at 0 1.2 360)
+			(layer "F.Fab")
+			(hide yes)
+			(effects
+				(font
+					(size 1 1)
+					(thickness 0.15)
+				)
+			)
+		)
+		(property "Footprint" "NetTie:NetTie-2_SMD_Pad0.5mm"
+			(at 0 0 180)
+			(unlocked yes)
+			(layer "F.Fab")
+			(hide yes)
+			(effects
+				(font
+					(size 1.27 1.27)
+					(thickness 0.15)
+				)
+			)
+		)
+		(property "Datasheet" ""
+			(at 0 0 180)
+			(unlocked yes)
+			(layer "F.Fab")
+			(hide yes)
+			(effects
+				(font
+					(size 1.27 1.27)
+					(thickness 0.15)
+				)
+			)
+		)
+		(property "Description" "Net tie, 2 pins"
+			(at 0 0 180)
+			(unlocked yes)
+			(layer "F.Fab")
+			(hide yes)
+			(effects
+				(font
+					(size 1.27 1.27)
+					(thickness 0.15)
+				)
+			)
+		)
+		(property ki_fp_filters "Net*Tie*")
+		(sheetname "Root")
+		(sheetfile "openautolab.kicad_sch")
+		(attr exclude_from_pos_files exclude_from_bom allow_missing_courtyard)
+		(net_tie_pad_groups "1, 2")
+		(fp_poly
+			(pts
+				(xy -0.5 -0.25) (xy 0.5 -0.25) (xy 0.5 0.25) (xy -0.5 0.25)
+			)
+			(stroke
+				(width 0)
+				(type solid)
+			)
+			(fill solid)
+			(layer "F.Cu")
+		)
+		(pad "1" smd circle
+			(at -0.5 0 180)
+			(size 0.5 0.5)
+			(layers "F.Cu")
+			(net 70 "GNDPWR")
+			(pinfunction "1")
+			(pintype "passive")
+		)
+		(pad "2" smd circle
+			(at 0.5 0 180)
+			(size 0.5 0.5)
+			(layers "F.Cu")
+			(net 28 "GND")
+			(pinfunction "2")
+			(pintype "passive")
+		)
+	)
 	(footprint "TerminalBlock_Phoenix:TerminalBlock_Phoenix_PT-1,5-2-3.5-H_1x02_P3.50mm_Horizontal"
 		(layer "F.Cu")
@@
 			(layers "F.Cu" "F.Paste" "F.Mask")
 			(roundrect_rratio 0.25)
-			(net 28 "GND")
+			(net 70 "GNDPWR")
 			(pinfunction "S")
 			(pintype "passive")
@@
 			(layers "F.Cu" "F.Paste" "F.Mask")
 			(roundrect_rratio 0.25)
-			(net 28 "GND")
+			(net 70 "GNDPWR")
 			(pintype "passive")
 		)
@@
 			(layers "F.Cu" "F.Paste" "F.Mask")
 			(roundrect_rratio 0.25)
-			(net 28 "GND")
+			(net 70 "GNDPWR")
 			(pintype "passive")
 		)
@@
 			(layers "F.Cu" "F.Paste" "F.Mask")
 			(roundrect_rratio 0.25)
-			(net 28 "GND")
+			(net 70 "GNDPWR")
 			(pinfunction "S")
 			(pintype "passive")
@@
 			(layers "F.Cu" "F.Paste" "F.Mask")
 			(roundrect_rratio 0.25)
-			(net 28 "GND")
+			(net 70 "GNDPWR")
 			(pintype "passive")
 		)
@@
 			(layers "F.Cu" "F.Paste" "F.Mask")
 			(roundrect_rratio 0.25)
-			(net 28 "GND")
+			(net 70 "GNDPWR")
 			(pinfunction "S")
 			(pintype "passive")
@@
 			(layers "F.Cu" "F.Paste" "F.Mask")
 			(roundrect_rratio 0.25)
-			(net 28 "GND")
+			(net 70 "GNDPWR")
 			(pinfunction "GND")
 			(pintype "power_in")
@@
 			(property pad_prop_heatsink)
 			(layers "F.Cu" "F.Mask")
-			(net 28 "GND")
+			(net 70 "GNDPWR")
 			(pinfunction "PAD")
 			(pintype "power_in")
@@
 			(layers "F.Cu" "F.Paste" "F.Mask")
 			(roundrect_rratio 0.1)
-			(net 28 "GND")
+			(net 70 "GNDPWR")
 			(pintype "passive")
 		)
@@
 			(layers "F.Cu" "F.Paste" "F.Mask")
 			(roundrect_rratio 0.25)
-			(net 28 "GND")
+			(net 70 "GNDPWR")
 			(pinfunction "S")
 			(pintype "passive")
@@
 			(layers "F.Cu" "F.Paste" "F.Mask")
 			(roundrect_rratio 0.25)
-			(net 28 "GND")
+			(net 70 "GNDPWR")
 			(pinfunction "S")
 			(pintype "passive")
@@
 			(layers "*.Cu" "*.Mask")
 			(remove_unused_layers no)
-			(net 28 "GND")
+			(net 70 "GNDPWR")
 			(pinfunction "Pin_1")
 			(pintype "passive")
@@
 			(layers "F.Cu" "F.Paste" "F.Mask")
 			(roundrect_rratio 0.25)
-			(net 28 "GND")
+			(net 70 "GNDPWR")
 			(pinfunction "S")
 			(pintype "passive")
@@
 			(layers "F.Cu" "F.Paste" "F.Mask")
 			(roundrect_rratio 0.25)
-			(net 28 "GND")
+			(net 70 "GNDPWR")
 			(pintype "passive")
 		)
@@
 			(layers "F.Cu" "F.Paste" "F.Mask")
 			(roundrect_rratio 0.25)
-			(net 28 "GND")
+			(net 70 "GNDPWR")
 			(pintype "passive")
 		)
@@
 			(layers "F.Cu" "F.Paste" "F.Mask")
 			(roundrect_rratio 0.25)
-			(net 28 "GND")
+			(net 70 "GNDPWR")
 			(pintype "passive")
 		)
@@
 			(layers "F.Cu" "F.Paste" "F.Mask")
 			(roundrect_rratio 0.25)
-			(net 28 "GND")
+			(net 70 "GNDPWR")
 			(pintype "passive")
 		)
@@
 			(layers "F.Cu" "F.Paste" "F.Mask")
 			(roundrect_rratio 0.25)
-			(net 28 "GND")
+			(net 70 "GNDPWR")
 			(pintype "passive")
 		)
@@
 			(layers "F.Cu" "F.Paste" "F.Mask")
 			(roundrect_rratio 0.25)
-			(net 28 "GND")
+			(net 70 "GNDPWR")
 			(pinfunction "S")
 			(pintype "passive")
@@
 			(layers "F.Cu" "F.Paste" "F.Mask")
 			(roundrect_rratio 0.25)
-			(net 28 "GND")
+			(net 70 "GNDPWR")
 			(pinfunction "S")
 			(pintype "passive")
@@
 			(layers "F.Cu" "F.Paste" "F.Mask")
 			(roundrect_rratio 0.227273)
-			(net 28 "GND")
+			(net 70 "GNDPWR")
 			(pinfunction "GND")
 			(pintype "power_in")
@@
 			(layers "F.Cu" "F.Paste")
 			(roundrect_rratio 0.054945)
-			(net 28 "GND")
+			(net 70 "GNDPWR")
 			(pinfunction "GND")
 			(pintype "power_in")
@@
 			(layers "F.Cu" "F.Paste")
 			(roundrect_rratio 0.054945)
-			(net 28 "GND")
+			(net 70 "GNDPWR")
 			(pinfunction "GND")
 			(pintype "power_in")
@@
 			(layers "F.Cu" "F.Mask")
 			(roundrect_rratio 0.026596)
-			(net 28 "GND")
+			(net 70 "GNDPWR")
 			(pinfunction "GND")
 			(pintype "power_in")
@@
 			(layers "F.Cu" "F.Paste")
 			(roundrect_rratio 0.054945)
-			(net 28 "GND")
+			(net 70 "GNDPWR")
 			(pinfunction "GND")
 			(pintype "power_in")
@@
 			(layers "F.Cu" "F.Paste")
 			(roundrect_rratio 0.054945)
-			(net 28 "GND")
+			(net 70 "GNDPWR")
 			(pinfunction "GND")
 			(pintype "power_in")
@@
 			(layers "F.Cu" "F.Paste" "F.Mask")
 			(roundrect_rratio 0.227273)
-			(net 28 "GND")
+			(net 70 "GNDPWR")
 			(pinfunction "~{ON}/OFF")
 			(pintype "input")
@@
 			(layers "F.Cu" "F.Paste" "F.Mask")
 			(roundrect_rratio 0.25)
-			(net 28 "GND")
+			(net 70 "GNDPWR")
 			(pinfunction "S")
 			(pintype "passive")
@@
 			(layers "F.Cu" "F.Paste" "F.Mask")
 			(roundrect_rratio 0.25)
-			(net 28 "GND")
+			(net 70 "GNDPWR")
 			(pintype "passive")
 		)
@@
 			(layers "F.Cu" "F.Paste" "F.Mask")
 			(roundrect_rratio 0.25)
-			(net 28 "GND")
+			(net 70 "GNDPWR")
 			(pintype "passive")
 		)

Commit message: really prepared for routing
Parts:
- moved U3 1.50 mm to (68.1, 66.4)
Connections:
- U3 pad 18: unconnected-(U3-GND-Pad18) -> GND
- U3 pad 42: GND -> unconnected-(U3-GND-Pad42)
Changed lines of the file:
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@@
 	(net 57 "unconnected-(U3-SWCLK-Pad41)")
 	(net 58 "unconnected-(U3-GND-Pad3)")
-	(net 59 "unconnected-(U3-GND-Pad18)")
+	(net 59 "unconnected-(U3-GND-Pad42)")
 	(net 60 "unconnected-(U3-3V3-Pad36)")
 	(net 61 "unconnected-(U3-GND-Pad8)")
@@
 		(tags "net tie")
 		(property "Reference" "NT1"
-			(at 0 -1.2 360)
+			(at 0 -1.2 0)
 			(layer "F.SilkS")
 			(hide yes)
@@
 		)
 		(property "Value" "NetTie_2"
-			(at 0 1.2 360)
+			(at 0 1.2 0)
 			(layer "F.Fab")
 			(hide yes)
@@
 		(tags "resistor")
 		(property "Reference" "R15"
-			(at 0 -1.43 360)
+			(at 0 -1.43 0)
 			(layer "F.SilkS")
 			(effects
@@
 		)
 		(property "Value" "100"
-			(at 0 1.43 360)
+			(at 0 1.43 0)
 			(layer "F.Fab")
 			(effects
@@
 		)
 		(fp_text user "${REFERENCE}"
-			(at 0 0 360)
+			(at 0 0 0)
 			(layer "F.Fab")
 			(effects
@@
 		(tags "capacitor electrolytic")
 		(property "Reference" "C1"
-			(at 0 -6.2 360)
+			(at 0 -6.2 0)
 			(layer "F.SilkS")
 			(effects
@@
 		)
 		(property "Value" "200uf"
-			(at 0 6.2 360)
+			(at 0 6.2 0)
 			(layer "F.Fab")
 			(effects
@@
 		)
 		(property "LCSC" "C125977"
-			(at 0 0 360)
+			(at 0 0 0)
 			(layer "F.SilkS")
 			(hide yes)
@@
 		)
 		(fp_text user "${REFERENCE}"
-			(at 0 0 360)
+			(at 0 0 0)
 			(layer "F.Fab")
 			(effects
@@
 		(tags "Through hole socket strip THT 1x03 2.54mm single row")
 		(property "Reference" "J14"
-			(at 0 -2.77 360)
+			(at 0 -2.77 0)
 			(layer "F.SilkS")
 			(effects
@@
 		)
 		(property "Value" "SERVO"
-			(at 0 7.85 360)
+			(at 0 7.85 0)
 			(layer "F.Fab")
 			(effects
@@
 		(tags "Through hole socket strip THT 1x04 2.54mm single row")
 		(property "Reference" "J13"
-			(at 0 -2.77 360)
+			(at 0 -2.77 0)
 			(layer "F.SilkS")
 			(effects
@@
 		)
 		(property "Value" "HX711"
-			(at 0 10.39 360)
+			(at 0 10.39 0)
 			(layer "F.Fab")
 			(effects
@@
 	(footprint "RP-Pico:RPi_Pico_SMD_TH"
 		(layer "F.Cu")
-		(at 68.11 64.89 90)
+		(at 68.11 66.39 90)
 		(descr "Through hole straight pin header, 2x20, 2.54mm pitch, double rows")
 		(tags "Through hole pin header THT 2x20 2.54mm double row")
@@
 			(layers "*.Cu" "*.Mask")
 			(remove_unused_layers no)
-			(net 59 "unconnected-(U3-GND-Pad18)")
+			(net 28 "GND")
 			(pinfunction "GND")
 			(pintype "power_in")
@@
 			)
 			(layers "F.Cu" "F.Mask")
-			(net 59 "unconnected-(U3-GND-Pad18)")
+			(net 28 "GND")
 			(pinfunction "GND")
 			(pintype "power_in")
@@
 			(layers "*.Cu" "*.Mask")
 			(remove_unused_layers no)
-			(net 28 "GND")
+			(net 59 "unconnected-(U3-GND-Pad42)")
 			(pinfunction "GND")
 			(pintype "power_in")
@@
 			)
 			(layers "F.Cu" "F.Mask")
-			(net 28 "GND")
+			(net 59 "unconnected-(U3-GND-Pad42)")
 			(pinfunction "GND")
 			(pintype "power_in")
@@
 		(tags "resistor")
 		(property "Reference" "R16"
-			(at 0 -1.43 360)
+			(at 0 -1.43 0)
 			(layer "F.SilkS")
 			(effects
@@
 		)
 		(property "Value" "10k"
-			(at 0 1.43 360)
+			(at 0 1.43 0)
 			(layer "F.Fab")
 			(effects
@@
 		)
 		(fp_text user "${REFERENCE}"
-			(at 0 0 360)
+			(at 0 0 0)
 			(layer "F.Fab")
 			(effects
@@
 		)
 		(fp_text user "${REFERENCE}"
-			(at 0 3.81 360)
+			(at 0 3.81 0)
 			(layer "F.Fab")
 			(effects

Commit message: routing done
Parts:
- moved R17 1.56 mm to (128.2, 54.5)
- moved R18 1.56 mm to (128.2, 52.5)
- moved C1 1.56 mm to (118.0, 63.5)
- moved C2 1.56 mm to (105.3, 59.5)
- moved C3 1.56 mm to (120.5, 50.5)
- moved D1 1.56 mm to (108.2, 81.5)
- moved D2 1.56 mm to (100.5, 46.5)
- moved D3 1.56 mm to (92.0, 46.5)
- moved D4 1.56 mm to (83.5, 46.5)
- moved D5 1.56 mm to (75.0, 46.5)
- moved D6 1.56 mm to (66.5, 46.5)
- moved D7 1.56 mm to (109.0, 46.5)
- moved D8 1.56 mm to (58.0, 46.5)
- moved J1 1.56 mm to (96.8, 39.8)
- moved J10 1.56 mm to (126.4, 42.5)
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Routing:
- net +12V: track 0.00 -> 276.5 mm
- net GNDPWR: track 0.00 -> 242.2 mm, vias 0 -> 2
- net GND: track 0.00 -> 178.0 mm
- net +5V: track 0.00 -> 163.1 mm, vias 0 -> 4
- net Net-(U3-GPIO2): track 0.00 -> 90.3 mm, vias 0 -> 1
- net Net-(J13-Pin_3): track 0.00 -> 83.2 mm
- net Net-(J13-Pin_2): track 0.00 -> 82.9 mm
- net Net-(U3-GPIO22): track 0.00 -> 80.1 mm, vias 0 -> 1
- net Net-(U3-GPIO20): track 0.00 -> 77.3 mm, vias 0 -> 1
- net Net-(U3-GPIO21): track 0.00 -> 71.8 mm, vias 0 -> 1
- net Net-(U3-GPIO5): track 0.00 -> 63.5 mm, vias 0 -> 1
- net Net-(U3-GPIO4): track 0.00 -> 55.3 mm, vias 0 -> 1
- net Net-(J14-Pin_3): track 0.00 -> 53.7 mm
- net Net-(U3-GPIO6): track 0.00 -> 50.6 mm, vias 0 -> 2
- net Net-(U3-GPIO11): track 0.00 -> 47.2 mm
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- added copper zone on F.Cu, net GNDPWR
