File: main_board/openautolab.kicad_sch (KiCad schematic)
At the start: 63 parts, among them J1 GP7, J10 FILTER_PUMP, J11 FILTER_SENSOR, J12 PWR_IN, J13 HX711, J14 SERVO, J15 Display, J2 GP6, J3 GP5, J4 GP4, J5 GP3, J6 GP2, J7 GP1, J8 GP0, J9 PUMP, Q1 TSM2302CX, Q2 TSM2302CX, Q3 TSM2302CX, Q4 TSM2302CX, Q5 TSM2302CX, Q6 TSM2302CX, Q7 TSM2302CX, Q8 TSM2302CX, Q9 TSM2302CX, SW0 GP20, SW1 GP21, SW2 GP22, SW3 SW_DPST_x2, U2 LM2575-5.0BT, U3 Pico, U4 A4950E

Commit message: prepare for routing
Parts:
- added NT1: NetTie_2, NetTie:NetTie-2_SMD_Pad0.5mm, symbol Device:NetTie_2
Connections:
- net GND: now also NT1.2; no longer C1.2, C3.2, J12.1 (Pin_1), Q1.2 (S), Q2.2 (S), Q3.2 (S), Q4.2 (S), Q5.2 (S), Q6.2 (S), Q7.2 (S), Q8.2 (S), Q9.2 (S), R10.2, R12.2, R14.2, R16.2, R18.2, R2.2, R4.2, R6.2, R8.2, U2.3 (GND), U2.5 (~{ON}/OFF), U4.1 (GND), U4.9 (PAD)
- new net GNDPWR: C1.2, C3.2, J12.1 (Pin_1), NT1.1, Q1.2 (S), Q2.2 (S), Q3.2 (S), Q4.2 (S), Q5.2 (S), Q6.2 (S), Q7.2 (S), Q8.2 (S), Q9.2 (S), R10.2, R12.2, R14.2, R16.2, R18.2, R2.2, R4.2, R6.2, R8.2, U2.3 (GND), U2.5 (~{ON}/OFF), U4.1 (GND), U4.9 (PAD)
Other:
- moved on the sheet: C1
Changed lines of the file:
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@@
 	)
 	(junction
-		(at 109.22 172.72)
-		(diameter 0)
-		(color 0 0 0 0)
-	)
-	(junction
 		(at 149.86 177.8)
 		(diameter 0)
@@
 	)
 	(junction
-		(at 113.03 185.42)
+		(at 138.43 26.67)
 		(diameter 0)
 		(color 0 0 0 0)
 	)
 	(junction
-		(at 138.43 26.67)
+		(at 273.05 30.48)
 		(diameter 0)
 		(color 0 0 0 0)
 	)
 	(junction
-		(at 273.05 30.48)
+		(at 113.03 185.42)
 		(diameter 0)
 		(color 0 0 0 0)
@@
 	)
 	(junction
-		(at 139.7 177.8)
+		(at 139.7 185.42)
 		(diameter 0)
 		(color 0 0 0 0)
 	)
 	(junction
-		(at 139.7 185.42)
+		(at 139.7 177.8)
 		(diameter 0)
 		(color 0 0 0 0)
@@
 	)
 	(junction
-		(at 207.01 31.75)
+		(at 125.73 185.42)
 		(diameter 0)
 		(color 0 0 0 0)
 	)
 	(junction
-		(at 125.73 185.42)
+		(at 207.01 31.75)
 		(diameter 0)
 		(color 0 0 0 0)
@@
 	)
 	(junction
-		(at 109.22 185.42)
-		(diameter 0)
-		(color 0 0 0 0)
-	)
-	(junction
 		(at 105.41 31.75)
 		(diameter 0)
@@
 	)
 	(junction
+		(at 107.95 172.72)
+		(diameter 0)
+		(color 0 0 0 0)
+	)
+	(junction
 		(at 53.34 24.13)
 		(diameter 0)
@@
 	)
 	(junction
+		(at 107.95 185.42)
+		(diameter 0)
+		(color 0 0 0 0)
+	)
+	(junction
 		(at 34.29 137.16)
 		(diameter 0)
@@
 	(wire
 		(pts
-			(xy 54.61 31.75) (xy 54.61 33.02)
+			(xy 125.73 182.88) (xy 125.73 185.42)
 		)
 		(stroke
@@
 	(wire
 		(pts
-			(xy 163.83 24.13) (xy 162.56 24.13)
+			(xy 54.61 31.75) (xy 54.61 33.02)
 		)
 		(stroke
@@
 	(wire
 		(pts
-			(xy 180.34 31.75) (xy 181.61 31.75)
+			(xy 163.83 24.13) (xy 162.56 24.13)
 		)
 		(stroke
@@
 	(wire
 		(pts
-			(xy 113.03 36.83) (xy 113.03 41.91)
+			(xy 180.34 31.75) (xy 181.61 31.75)
 		)
 		(stroke
@@
 	(wire
 		(pts
-			(xy 104.14 19.05) (xy 104.14 24.13)
+			(xy 113.03 36.83) (xy 113.03 41.91)
 		)
 		(stroke
@@
 	(wire
 		(pts
-			(xy 109.22 172.72) (xy 113.03 172.72)
+			(xy 104.14 19.05) (xy 104.14 24.13)
 		)
 		(stroke
@@
 	(wire
 		(pts
-			(xy 109.22 172.72) (xy 109.22 175.26)
+			(xy 107.95 172.72) (xy 107.95 175.26)
 		)
 		(stroke
@@
 	(wire
 		(pts
-			(xy 101.6 185.42) (xy 109.22 185.42)
+			(xy 101.6 185.42) (xy 107.95 185.42)
 		)
 		(stroke
@@
 	(wire
 		(pts
+			(xy 134.62 185.42) (xy 139.7 185.42)
+		)
+		(stroke
+			(width 0)
+			(type default)
+		)
+	)
+	(wire
+		(pts
 			(xy 53.34 31.75) (xy 54.61 31.75)
 		)
@@
 	(wire
 		(pts
+			(xy 107.95 185.42) (xy 113.03 185.42)
+		)
+		(stroke
+			(width 0)
+			(type default)
+		)
+	)
+	(wire
+		(pts
 			(xy 130.81 31.75) (xy 130.81 33.02)
 		)
@@
 	(wire
 		(pts
-			(xy 109.22 182.88) (xy 109.22 185.42)
-		)
-		(stroke
-			(width 0)
-			(type default)
-		)
-	)
-	(wire
-		(pts
 			(xy 105.41 31.75) (xy 105.41 33.02)
 		)
@@
 	(wire
 		(pts
-			(xy 101.6 172.72) (xy 109.22 172.72)
+			(xy 101.6 172.72) (xy 107.95 172.72)
 		)
 		(stroke
@@
 	(wire
 		(pts
+			(xy 125.73 185.42) (xy 129.54 185.42)
+		)
+		(stroke
+			(width 0)
+			(type default)
+		)
+	)
+	(wire
+		(pts
 			(xy 36.83 137.16) (xy 34.29 137.16)
 		)
@@
 	(wire
 		(pts
+			(xy 107.95 182.88) (xy 107.95 185.42)
+		)
+		(stroke
+			(width 0)
+			(type default)
+		)
+	)
+	(wire
+		(pts
 			(xy 36.83 26.67) (xy 36.83 24.13)
 		)
@@
 	(wire
 		(pts
+			(xy 113.03 177.8) (xy 113.03 185.42)
+		)
+		(stroke
+			(width 0)
+			(type default)
+		)
+	)
+	(wire
+		(pts
 			(xy 158.75 111.76) (xy 179.07 111.76)
 		)
@@
 	(wire
 		(pts
+			(xy 107.95 172.72) (xy 113.03 172.72)
+		)
+		(stroke
+			(width 0)
+			(type default)
+		)
+	)
+	(wire
+		(pts
 			(xy 158.75 99.06) (xy 182.88 99.06)
 		)
@@
 	(wire
 		(pts
-			(xy 109.22 185.42) (xy 113.03 185.42)
-		)
-		(stroke
-			(width 0)
-			(type default)
-		)
-	)
-	(wire
-		(pts
-			(xy 125.73 185.42) (xy 125.73 182.88)
-		)
-		(stroke
-			(width 0)
-			(type default)
-		)
-	)
-	(wire
-		(pts
 			(xy 24.13 101.6) (xy 24.13 120.65)
 		)
@@
 	(wire
 		(pts
-			(xy 113.03 177.8) (xy 113.03 185.42)
-		)
-		(stroke
-			(width 0)
-			(type default)
-		)
-	)
-	(wire
-		(pts
 			(xy 182.88 93.98) (xy 182.88 104.14)
 		)
@@
 	(wire
 		(pts
-			(xy 125.73 185.42) (xy 139.7 185.42)
-		)
-		(stroke
-			(width 0)
-			(type default)
-		)
-	)
-	(wire
-		(pts
 			(xy 77.47 115.57) (xy 76.2 115.57)
 		)
@@
 	)
 	(symbol
+		(lib_id "Device:NetTie_2")
+		(at 132.08 185.42 0)
+		(unit 1)
+		(exclude_from_sim no)
+		(in_bom no)
+		(on_board yes)
+		(dnp no)
+		(fields_autoplaced yes)
+		(property "Reference" "NT1"
+			(at 132.08 180.34 0)
+			(effects
+				(font
+					(size 1.27 1.27)
+				)
+			)
+		)
+		(property "Value" "NetTie_2"
+			(at 132.08 182.88 0)
+			(effects
+				(font
+					(size 1.27 1.27)
+				)
+			)
+		)
+		(property "Footprint" "NetTie:NetTie-2_SMD_Pad0.5mm"
+			(at 132.08 185.42 0)
+			(effects
+				(font
+					(size 1.27 1.27)
+				)
+				(hide yes)
+			)
+		)
+		(property "Datasheet" "~"
+			(at 132.08 185.42 0)
+			(effects
+				(font
+					(size 1.27 1.27)
+				)
+				(hide yes)
+			)
+		)
+		(property "Description" "Net tie, 2 pins"
+			(at 132.08 185.42 0)
+			(effects
+				(font
+					(size 1.27 1.27)
+				)
+				(hide yes)
+			)
+		)
+		(pin "1"
+		)
+		(pin "2"
+		)
+		(instances
+			(project ""
+				(path "/cfdd5521-a8c1-4ce8-a79b-bc50281bd389"
+					(reference "NT1")
+					(unit 1)
+				)
+			)
+		)
+	)
+	(symbol
 		(lib_id "power:GNDPWR")
 		(at 87.63 43.18 0)
@@
 		)
 		(property "Value" "1N5819WS"
-			(at 128.27 184.15 90)
+			(at 137.16 186.944 90)
 			(effects
 				(font
@@
 	(symbol
 		(lib_id "Device:C_Polarized")
-		(at 109.22 179.07 0)
+		(at 107.95 179.07 0)
 		(unit 1)
 		(exclude_from_sim no)
@@
 		(dnp no)
 		(property "Reference" "C1"
-			(at 102.87 177.8 0)
+			(at 101.6 177.8 0)
 			(effects
 				(font
@@
 		)
 		(property "Value" "200uf"
-			(at 101.092 180.34 0)
+			(at 99.822 180.34 0)
 			(effects
 				(font
@@
 		)
 		(property "Footprint" "Capacitor_SMD:CP_Elec_10x10"
-			(at 110.1852 182.88 0)
+			(at 108.9152 182.88 0)
 			(effects
 				(font
@@
 		)
 		(property "Datasheet" "~"
-			(at 109.22 179.07 0)
+			(at 107.95 179.07 0)
 			(effects
 				(font
@@
 		)
 		(property "Description" ""
-			(at 109.22 179.07 0)
+			(at 107.95 179.07 0)
 			(effects
 				(font
@@
 		)
 		(property "LCSC" "C125977"
-			(at 0 358.14 0)
+			(at -1.27 358.14 0)
 			(effects
 				(font

Commit message: really prepared for routing
Parts:
- SW3: footprint Connector_PinHeader_2.54mm:PinHeader_1x02_P2.54mm_Vertical -> easyeda2kicad:SW-SMD_6P-L5.8-W5.8-P2.00-LS8.0_YTSPS-22E58LM
Connections:
- net GND: now also U3.18 (GND); no longer U3.42 (GND)
Other:
- moved on the sheet: J9

Commit message: minor routing-related stuff
Parts:
- SW3: footprint easyeda2kicad:SW-SMD_6P-L5.8-W5.8-P2.00-LS8.0_YTSPS-22E58LM -> JLCPCB:SW-SMD_6P-L5.8-W5.8-P2.00-LS8.0_YTSPS-22E58LM
- U3: footprint RP-Pico:RPi_Pico_SMD_TH -> RPi Pico:RPi_Pico_SMD_TH
Changed lines of the file:
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@@
 			)
 		)
-		(property "Footprint" "easyeda2kicad:SW-SMD_6P-L5.8-W5.8-P2.00-LS8.0_YTSPS-22E58LM"
+		(property "Footprint" "JLCPCB:SW-SMD_6P-L5.8-W5.8-P2.00-LS8.0_YTSPS-22E58LM"
 			(at 243.84 25.4 0)
 			(effects
@@
 			)
 		)
-		(property "Footprint" "RP-Pico:RPi_Pico_SMD_TH"
+		(property "Footprint" "RPi Pico:RPi_Pico_SMD_TH"
 			(at 140.97 90.17 90)
 			(effects
